Commit message: Update robot code from Raspberry Pi

File: src/my_robot_description/urdf/mobile_base.xacro (robot description, xacro)
@@ -1,9 +1,10 @@
 <?xml version="1.0"?>
 <robot xmlns:xacro="http://www.ros.org/wiki/xacro">
-    <xacro:property name="base_length" value="0.6" />
-    <xacro:property name="base_width" value="0.4" />
-    <xacro:property name="base_height" value="0.2" />
-    <xacro:property name="wheel_radius" value="0.1" />
-    <xacro:property name="wheel_length" value="0.05" />
+    <xacro:property name="base_length" value="0.233" />
+    <xacro:property name="base_width" value="0.261" />
+    <xacro:property name="base_height" value="0.120" />
+    <xacro:property name="wheel_radius" value="0.036" />
+    <xacro:property name="wheel_length" value="0.040" />
+    <xacro:property name="wheel_separation" value="0.235" />
     <link name="base_footprint" />
     <link name="base_link">
@@ -70,5 +71,5 @@
         <parent link="base_link" />
         <child link="right_wheel_link" />
-        <origin xyz="${-base_length / 4.0} ${-(base_width + wheel_length) / 2.0} 0" rpy="0 0 0" />
+        <origin xyz="${-wheel_separation / 2.0} ${-(base_width + wheel_length) / 2.0} 0" rpy="0 0 0" />
         <axis xyz="0 1 0" />
     </joint>
@@ -76,5 +77,5 @@
         <parent link="base_link" />
         <child link="left_wheel_link" />
-        <origin xyz="${-base_length / 4.0} ${(base_width + wheel_length) / 2.0} 0" rpy="0 0 0" />
+        <origin xyz="${wheel_separation / 2.0} ${(base_width + wheel_length) / 2.0} 0" rpy="0 0 0" />
         <axis xyz="0 1 0" />
     </joint>

Commit message: Rev 1

File: src/my_robot_description/urdf/mobile_base.xacro (robot description, xacro)
@@ -7,4 +7,5 @@
     <xacro:property name="wheel_length" value="0.040" />
     <xacro:property name="wheel_separation" value="0.235" />
+    <xacro:property name="wheel_x_offset" value="0.0" />
     <link name="base_footprint" />
     <link name="base_link">
@@ -71,11 +72,11 @@
         <parent link="base_link" />
         <child link="right_wheel_link" />
-        <origin xyz="${-wheel_separation / 2.0} ${-(base_width + wheel_length) / 2.0} 0" rpy="0 0 0" />
-        <axis xyz="0 1 0" />
+        <origin xyz="${wheel_x_offset} ${-wheel_separation / 2.0} 0" rpy="0 0 0" />
+	<axis xyz="0 1 0" />
     </joint>
     <joint name="base_left_wheel_joint" type="continuous">
         <parent link="base_link" />
         <child link="left_wheel_link" />
-        <origin xyz="${wheel_separation / 2.0} ${(base_width + wheel_length) / 2.0} 0" rpy="0 0 0" />
+        <origin xyz="${wheel_x_offset} ${wheel_separation / 2.0} 0" rpy="0 0 0" />
         <axis xyz="0 1 0" />
     </joint>

Commit message: Rev 2

File: src/my_robot_description/urdf/mobile_base.xacro (robot description, xacro)
@@ -1,6 +1,6 @@
 <?xml version="1.0"?>
 <robot xmlns:xacro="http://www.ros.org/wiki/xacro">
-    <xacro:property name="base_length" value="0.233" />
-    <xacro:property name="base_width" value="0.261" />
+    <xacro:property name="base_length" value="0.261" />
+    <xacro:property name="base_width" value="0.233" />
     <xacro:property name="base_height" value="0.120" />
     <xacro:property name="wheel_radius" value="0.036" />
