Commit message: Rev 3

File: src/my_robot_description/urdf/lidar.xacro (robot description, xacro)
@@ -21,5 +21,5 @@
         <parent link="base_link"/>
         <child link="laser_link"/>
-        <origin xyz="-${base_length / 3.0} 0 ${base_height + (laser_length / 2.0)}" rpy="0 0 ${pi}"/>
+        <origin xyz="0 0 ${base_height + (laser_length / 2.0)}" rpy="0 0 0"/>
     </joint>
     <gazebo reference="laser_link">
